File: pcb/oscilloscope.brd (EAGLE design)
At the start: 60.6 x 128.5 mm, 37 parts, among them J1 35PM1, J2 35PM1, J3 35PM1, J4 35PM1, J5 35PM1, J6 35PM1, J7 35PM1, J8 35PM1, M1 ESP32, SW1 EN12-HS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

Commit message: Updating PCB to rev B
Parts:
- added C10, C5, C6, C7, C8, C9: 47nF, rcl:C0805
- added C11, C4: (no value), rcl:C0805
- added R19, R20, R21, R22, R23: 10k, rcl:R0805
- added U4: ESP-PSRAM64, artysynth:SOIC-8
- added U5: 74HC14, artysynth:SOIC127P600X175-14N
- R13, R14: value (none) -> 10k
- moved R14 10.2 mm to (40.5, 13.5), turned to 0 degrees
- moved R13 7.55 mm to (21.8, 25.1), turned to 180 degrees
- moved R15 3.02 mm to (13.8, 115.6)
- moved R17 3.02 mm to (8.76, 115.6)
- moved R16 3.02 mm to (13.8, 112.5)
- moved R18 3.02 mm to (8.76, 112.5)
Connections:
- removed net ADC2_CH8: M1.X8
- new net ENC1_A_I: C5.1, R21.2, SW1.A, U5.3
- new net ENC1_B_I: C6.1, R20.2, SW1.B, U5.1
- new net ENC2_A_I: C8.1, R23.2, SW2.A, U5.11
- new net ENC2_B_I: C9.1, R22.2, SW2.B, U5.9
- new net SPIRAM_CE: M1.X26, R19.2, U4.1
- new net SPIRAM_CLK: M1.X19, U4.6
- new net SPIRAM_D0: M1.X20, U4.5
- new net SPIRAM_D1: M1.X21, U4.2
- new net SPIRAM_D2: M1.X15, U4.3
- new net SPIRAM_D3: M1.X16, U4.7
- new net SW1_I: C7.1, R13.2, SW1.D, U5.5
- new net SW2_I: C10.1, R14.2, SW2.D, U5.13
- net +3V3: now also C11.1, C4.2, R19.1, R20.1, R21.1, R22.1, R23.1, U4.8, U5.14
- net ENC1_A: now also M1.X25, U5.4; no longer M1.X26, SW1.A
- net ENC1_B: now also M1.X24, U5.2; no longer M1.X25, SW1.B
- net ENC2_A: now also M1.X12, U5.10; no longer M1.X14, SW2.A
- net ENC2_B: now also M1.X14, U5.8; no longer M1.X12, SW2.B
- net GND: now also C10.2, C11.2, C4.1, C5.2, C6.2, C7.2, C8.2, C9.2, U4.4, U5.7
- net SW1: now also M1.X8, U5.6; no longer M1.X24, R13.2, SW1.D
- net SW2: now also U5.12; no longer R14.2, SW2.D
Routing:
- net SPIRAM_CE: track 0.00 -> 33.5 mm
- net ENC1_B_I: track 0.00 -> 28.5 mm
- net ENC1_A_I: track 0.00 -> 27.1 mm
- net ENC2_B_I: track 0.00 -> 26.4 mm
- net ENC2_A_I: track 0.00 -> 26.1 mm
- net +3V3: track 35.5 -> 56.8 mm, vias 9 -> 17
- net SW1: track 73.5 -> 93.4 mm, vias 0 -> 1
- net ENC2_A: track 115.5 -> 98.6 mm, vias 0 -> 1
- net SPIRAM_D1: track 0.00 -> 16.8 mm, vias 0 -> 1
- net SPIRAM_D2: track 0.00 -> 15.7 mm, vias 0 -> 1
- net SPIRAM_CLK: track 0.00 -> 14.0 mm
- net SPIRAM_D3: track 0.00 -> 12.9 mm, vias 0 -> 1
- net ENC2_B: track 108.7 -> 96.1 mm, vias 0 -> 1
- net SW2_I: track 0.00 -> 12.5 mm
- net SPIRAM_D0: track 0.00 -> 11.2 mm
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- added copper zone on layer 1, net GND
Other:
- board text added: "OSCILLOSCOPE MODULE Rev B / Jan 2021 Brian Boucher"
- board text removed: "OSCILLOSCOPE MODULE Rev A / Jan 2021 Brian Boucher"
